File: ESP-WROOM-32-Breakout.sch (EAGLE design)
At the start: 29 parts, among them U3 ESP-WROOM-32

Commit message: Add files via upload
Parts:
- removed R5: 150K, hari:RESISTOR0402
- removed R6: 47K, hari:RESISTOR0402
- added R8: 150K, rcl:R-EU_R0603
- added R9: 47K, rcl:R-EU_R0603
Connections:
- net GND: now also R9.1; no longer R6.1
- net N$4: now also R8.2, R9.2; no longer R5.2, R6.2
- net VCC: now also R8.1; no longer R5.1
Changed lines of the file:
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@@
 <part name="U$2" library="hari" deviceset="TPS82140" device=""/>
 <part name="GND9" library="SparkFun-Aesthetics" deviceset="GND" device=""/>
-<part name="R5" library="hari" deviceset="RESISTOR" device="0402" value="150K"/>
-<part name="R6" library="hari" deviceset="RESISTOR" device="0402" value="47K"/>
 <part name="GND11" library="SparkFun-Aesthetics" deviceset="GND" device=""/>
 <part name="C7" library="hari" deviceset="CAP_CERAMIC" device="0603" value="3n3"/>
@@
 <part name="C10" library="rcl" deviceset="C-EU" device="C0603" value="10u"/>
 <part name="JP4" library="hari" deviceset="HEADER-1X1" device="ROUND"/>
+<part name="R8" library="rcl" deviceset="R-EU_" device="R0603" value="150K"/>
+<part name="R9" library="rcl" deviceset="R-EU_" device="R0603" value="47K"/>
 </parts>
 <sheets>
@@
 </instance>
 <instance part="GND9" gate="1" x="218.44" y="129.54"/>
-<instance part="R5" gate="G$1" x="243.84" y="139.7" rot="R90"/>
-<instance part="R6" gate="G$1" x="248.92" y="144.78" rot="R180"/>
 <instance part="GND11" gate="1" x="254" y="134.62"/>
 <instance part="C7" gate="G$1" x="236.22" y="154.94" rot="R90"/>
@@
 <instance part="C10" gate="G$1" x="238.76" y="116.84"/>
 <instance part="JP4" gate="G$1" x="91.44" y="40.64" rot="R270"/>
+<instance part="R8" gate="G$1" x="243.84" y="139.7" rot="R90"/>
+<instance part="R9" gate="G$1" x="248.92" y="144.78" rot="R180"/>
 </instances>
 <busses>
@@
 </segment>
 <segment>
-<pinref part="R6" gate="G$1" pin="1"/>
 <pinref part="GND11" gate="1" pin="GND"/>
 <wire x1="254" y1="137.16" x2="254" y2="144.78" width="0.1524" layer="91"/>
+<pinref part="R9" gate="G$1" pin="1"/>
 </segment>
 <segment>
@@
 <wire x1="231.14" y1="119.38" x2="231.14" y2="134.62" width="0.1524" layer="91"/>
 <junction x="218.44" y="119.38"/>
-<pinref part="R5" gate="G$1" pin="1"/>
 <wire x1="231.14" y1="134.62" x2="231.14" y2="139.7" width="0.1524" layer="91"/>
 <wire x1="231.14" y1="134.62" x2="243.84" y2="134.62" width="0.1524" layer="91"/>
@@
 <wire x1="231.14" y1="119.38" x2="238.76" y2="119.38" width="0.1524" layer="91"/>
 <junction x="231.14" y="119.38"/>
+<pinref part="R8" gate="G$1" pin="1"/>
 </segment>
 <segment>
@@
 <segment>
 <pinref part="U$2" gate="G$1" pin="FB"/>
-<pinref part="R5" gate="G$1" pin="2"/>
 <wire x1="231.14" y1="144.78" x2="243.84" y2="144.78" width="0.1524" layer="91"/>
-<pinref part="R6" gate="G$1" pin="2"/>
+<pinref part="R8" gate="G$1" pin="2"/>
+<pinref part="R9" gate="G$1" pin="2"/>
 <junction x="243.84" y="144.78"/>
 </segment>

Commit message: Add files via upload
moved led to pin 13, changed cap package C11 (now can accomodate tantalum B size e.g. 220uf 4V), remove thermals on some footprints for contiguous ground plane
Parts:
- removed C10: 10u, rcl:C-EUC0603
- added C11: (no value), SparkFun-Passives:CAPSMD
Connections:
- net GND: now also C11.2; no longer C10.2
- net IO13: now also LED1.A
- net IO15: no longer LED1.A
- net VCC: now also C11.1; no longer C10.1
Other:
- moved on the sheet: LED1, R7
Changed lines of the file:
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@@
 <part name="R7" library="rcl" deviceset="R-EU_" device="R0603" value="1K"/>
 <part name="GND13" library="SparkFun-Aesthetics" deviceset="GND" device=""/>
-<part name="C10" library="rcl" deviceset="C-EU" device="C0603" value="10u"/>
 <part name="JP4" library="hari" deviceset="HEADER-1X1" device="ROUND"/>
 <part name="R8" library="rcl" deviceset="R-EU_" device="R0603" value="150K"/>
 <part name="R9" library="rcl" deviceset="R-EU_" device="R0603" value="47K"/>
+<part name="C11" library="SparkFun-Passives" deviceset="CAP" device="SMD"/>
 </parts>
 <sheets>
@@
 <instance part="C8" gate="G$1" x="228.6" y="116.84"/>
 <instance part="C9" gate="G$1" x="205.74" y="116.84"/>
-<instance part="LED1" gate="G$1" x="66.04" y="35.56" rot="R270"/>
-<instance part="R7" gate="G$1" x="66.04" y="27.94" rot="R90"/>
-<instance part="GND13" gate="1" x="66.04" y="20.32"/>
-<instance part="C10" gate="G$1" x="238.76" y="116.84"/>
+<instance part="LED1" gate="G$1" x="53.34" y="38.1" rot="R270"/>
+<instance part="R7" gate="G$1" x="53.34" y="30.48" rot="R90"/>
+<instance part="GND13" gate="1" x="53.34" y="22.86"/>
 <instance part="JP4" gate="G$1" x="91.44" y="40.64" rot="R270"/>
 <instance part="R8" gate="G$1" x="243.84" y="139.7" rot="R90"/>
 <instance part="R9" gate="G$1" x="248.92" y="144.78" rot="R180"/>
+<instance part="C11" gate="G$1" x="238.76" y="114.3"/>
 </instances>
 <busses>
@@
 <pinref part="C8" gate="G$1" pin="2"/>
 <wire x1="218.44" y1="111.76" x2="228.6" y2="111.76" width="0.1524" layer="91"/>
-<pinref part="C10" gate="G$1" pin="2"/>
+<pinref part="C11" gate="G$1" pin="2"/>
 <wire x1="228.6" y1="111.76" x2="238.76" y2="111.76" width="0.1524" layer="91"/>
 <junction x="228.6" y="111.76"/>
@@
 <pinref part="C9" gate="G$1" pin="1"/>
 <junction x="205.74" y="119.38"/>
-<pinref part="C10" gate="G$1" pin="1"/>
 <wire x1="231.14" y1="119.38" x2="238.76" y2="119.38" width="0.1524" layer="91"/>
 <junction x="231.14" y="119.38"/>
 <pinref part="R8" gate="G$1" pin="1"/>
+<pinref part="C11" gate="G$1" pin="1"/>
 </segment>
 <segment>
@@
 <segment>
 <pinref part="JP1" gate="G$1" pin="2"/>
-<wire x1="33.02" y1="43.18" x2="45.72" y2="43.18" width="0.1524" layer="91"/>
+<wire x1="33.02" y1="43.18" x2="53.34" y2="43.18" width="0.1524" layer="91"/>
 <label x="43.18" y="43.18" size="1.778" layer="95"/>
+<pinref part="LED1" gate="G$1" pin="A"/>
 </segment>
 </net>
@@
 <segment>
 <pinref part="JP2" gate="G$1" pin="1"/>
-<wire x1="71.12" y1="40.64" x2="66.04" y2="40.64" width="0.1524" layer="91"/>
+<wire x1="71.12" y1="40.64" x2="60.96" y2="40.64" width="0.1524" layer="91"/>
 <label x="60.96" y="40.64" size="1.778" layer="95"/>
-<pinref part="LED1" gate="G$1" pin="A"/>
-<wire x1="66.04" y1="40.64" x2="60.96" y2="40.64" width="0.1524" layer="91"/>
-<junction x="66.04" y="40.64"/>
-</segment>
-</net>
+</segment>
+</net>
